Commit message: The Lidar sensor is integraeted and working!

File: description/rover.urdf.xacro (robot description, xacro)
@@ -3,3 +3,4 @@
     <xacro:include filename="rover_core.xacro" />
     <xacro:include filename="gazebo_controls.xacro" />
+    <xacro:include filename="lidar.xacro" />
 </robot>

File: description/rover_core.xacro (robot description, xacro)
@@ -13,4 +13,7 @@
     <material name="black">
         <color rgba="0 0 0 1" />
+    </material>
+    <material name="red">
+        <color rgba="1 0 0 1" />
     </material>
     <!-- BASE LINK -->
